File: Blinky/Blinky.kicad_sch (KiCad schematic)
At the start: 12 parts, among them IC1 PAM8303CBSC, J1 TP4056, J2 Battery Connector, J3 Speaker Connector, J4 USB_B_Micro, J5 Charging Notches, SW1 SW_Push, U1 ESP32-S2-WROVER

Commit message: bugfix
Connections:
- new net: 1k1.1, 2k1.2, IC1.3 (VDD), J1.5 (BAT), J2.1 (Pin_1), SW1.1, U1.2 (3V3), ZTS6156.1 (VDD)
- new net: J4.2 (D-), U1.22 (USB_D-)
- new net: J4.3 (D+), U1.23 (USB_D+)
- new net: U1.33 (IO39), ZTS6156.2 (OUTPUT)
- new net: IC1.4 (IN-), U1.25 (IO26)
- now unconnected: U1.10 (IO07), U1.11 (IO08), U1.12 (IO09), U1.13 (IO10), U1.14 (IO11), U1.15 (IO12), U1.16 (IO13), U1.17 (IO14), U1.18 (IO15), U1.19 (IO16), U1.20 (IO17), U1.21 (IO18), U1.24 (IO21), U1.27 (IO33), U1.28 (IO34), U1.29 (IO35), U1.3 (IO00), U1.30 (IO36), U1.31 (IO37), U1.32 (IO38), U1.4 (IO01), U1.41 (EN), U1.5 (IO02), U1.6 (IO03), U1.7 (IO04), U1.8 (IO05), U1.9 (IO06)
Changed lines of the file:
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@@
 (kicad_sch (version 20230121) (generator eeschema)
   (paper "A4")
-  (junction (at 130.81 96.52) (diameter 0) (color 0 0 0 0)
-  )
-  (junction (at 130.81 101.6) (diameter 0) (color 0 0 0 0)
-  )
   (junction (at 146.05 48.26) (diameter 0) (color 0 0 0 0)
   )
-  (junction (at 130.81 88.9) (diameter 0) (color 0 0 0 0)
-  )
   (junction (at 237.49 48.26) (diameter 0) (color 0 0 0 0)
   )
-  (junction (at 130.81 71.12) (diameter 0) (color 0 0 0 0)
-  )
-  (junction (at 130.81 86.36) (diameter 0) (color 0 0 0 0)
-  )
-  (junction (at 161.29 76.2) (diameter 0) (color 0 0 0 0)
-  )
-  (junction (at 130.81 93.98) (diameter 0) (color 0 0 0 0)
-  )
-  (junction (at 161.29 121.92) (diameter 0) (color 0 0 0 0)
-  )
-  (junction (at 130.81 53.34) (diameter 0) (color 0 0 0 0)
-  )
   (junction (at 146.05 143.51) (diameter 0) (color 0 0 0 0)
   )
-  (junction (at 130.81 68.58) (diameter 0) (color 0 0 0 0)
-  )
-  (junction (at 130.81 99.06) (diameter 0) (color 0 0 0 0)
-  )
-  (junction (at 130.81 81.28) (diameter 0) (color 0 0 0 0)
+  (junction (at 175.26 125.73) (diameter 0) (color 0 0 0 0)
   )
   (junction (at 146.05 113.03) (diameter 0) (color 0 0 0 0)
   )
-  (junction (at 161.29 88.9) (diameter 0) (color 0 0 0 0)
-  )
-  (junction (at 130.81 76.2) (diameter 0) (color 0 0 0 0)
-  )
-  (junction (at 130.81 91.44) (diameter 0) (color 0 0 0 0)
-  )
-  (junction (at 161.29 81.28) (diameter 0) (color 0 0 0 0)
-  )
-  (junction (at 161.29 83.82) (diameter 0) (color 0 0 0 0)
-  )
-  (junction (at 161.29 86.36) (diameter 0) (color 0 0 0 0)
-  )
-  (junction (at 130.81 55.88) (diameter 0) (color 0 0 0 0)
-  )
   (junction (at 172.72 52.07) (diameter 0) (color 0 0 0 0)
   )
-  (junction (at 161.29 96.52) (diameter 0) (color 0 0 0 0)
-  )
-  (junction (at 130.81 58.42) (diameter 0) (color 0 0 0 0)
-  )
-  (junction (at 161.29 91.44) (diameter 0) (color 0 0 0 0)
-  )
   (junction (at 130.81 123.19) (diameter 0) (color 0 0 0 0)
   )
-  (junction (at 130.81 63.5) (diameter 0) (color 0 0 0 0)
-  )
   (junction (at 254 73.66) (diameter 0) (color 0 0 0 0)
   )
-  (junction (at 130.81 83.82) (diameter 0) (color 0 0 0 0)
-  )
-  (junction (at 130.81 78.74) (diameter 0) (color 0 0 0 0)
-  )
-  (junction (at 161.29 93.98) (diameter 0) (color 0 0 0 0)
-  )
-  (junction (at 130.81 73.66) (diameter 0) (color 0 0 0 0)
-  )
-  (junction (at 161.29 73.66) (diameter 0) (color 0 0 0 0)
-  )
   (junction (at 237.49 49.53) (diameter 0) (color 0 0 0 0)
   )
-  (junction (at 130.81 60.96) (diameter 0) (color 0 0 0 0)
-  )
-  (junction (at 161.29 78.74) (diameter 0) (color 0 0 0 0)
-  )
   (junction (at 172.72 68.58) (diameter 0) (color 0 0 0 0)
   )
-  (junction (at 130.81 66.04) (diameter 0) (color 0 0 0 0)
-  )
   (wire (pts (xy 146.05 143.51) (xy 146.05 137.16))
     (stroke (width 0) (type default))
@@
     (stroke (width 0) (type default))
   )
-  (wire (pts (xy 130.81 55.88) (xy 130.81 58.42))
-    (stroke (width 0) (type default))
-  )
   (wire (pts (xy 254 39.37) (xy 237.49 39.37))
     (stroke (width 0) (type default))
   )
-  (wire (pts (xy 130.81 101.6) (xy 130.81 123.19))
-    (stroke (width 0) (type default))
-  )
-  (wire (pts (xy 130.81 96.52) (xy 130.81 99.06))
+  (wire (pts (xy 127 110.49) (xy 130.81 110.49))
     (stroke (width 0) (type default))
   )
@@
     (stroke (width 0) (type default))
   )
+  (wire (pts (xy 130.81 110.49) (xy 130.81 123.19))
+    (stroke (width 0) (type default))
+  )
+  (wire (pts (xy 171.45 88.9) (xy 171.45 125.73))
+    (stroke (width 0) (type default))
+  )
   (wire (pts (xy 237.49 48.26) (xy 237.49 49.53))
     (stroke (width 0) (type default))
@@
     (stroke (width 0) (type default))
   )
-  (wire (pts (xy 130.81 71.12) (xy 130.81 73.66))
-    (stroke (width 0) (type default))
-  )
   (wire (pts (xy 130.81 123.19) (xy 130.81 128.27))
     (stroke (width 0) (type default))
   )
-  (wire (pts (xy 130.81 86.36) (xy 130.81 88.9))
-    (stroke (width 0) (type default))
-  )
   (wire (pts (xy 237.49 52.07) (xy 172.72 52.07))
     (stroke (width 0) (type default))
@@
     (stroke (width 0) (type default))
   )
+  (wire (pts (xy 127 48.26) (xy 127 110.49))
+    (stroke (width 0) (type default))
+  )
   (wire (pts (xy 238.76 52.07) (xy 238.76 90.17))
     (stroke (width 0) (type default))
@@
     (stroke (width 0) (type default))
   )
+  (wire (pts (xy 163.83 121.92) (xy 97.79 121.92))
+    (stroke (width 0) (type default))
+  )
   (wire (pts (xy 161.29 143.51) (xy 157.48 143.51))
     (stroke (width 0) (type default))
   )
-  (wire (pts (xy 130.81 66.04) (xy 130.81 68.58))
-    (stroke (width 0) (type default))
-  )
   (wire (pts (xy 140.97 173.99) (xy 140.97 168.91))
     (stroke (width 0) (type default))
   )
-  (wire (pts (xy 130.81 91.44) (xy 130.81 93.98))
-    (stroke (width 0) (type default))
-  )
   (wire (pts (xy 97.79 121.92) (xy 97.79 128.27))
     (stroke (width 0) (type default))
@@
     (stroke (width 0) (type default))
   )
-  (wire (pts (xy 130.81 83.82) (xy 130.81 86.36))
-    (stroke (width 0) (type default))
-  )
-  (wire (pts (xy 130.81 53.34) (xy 130.81 55.88))
+  (wire (pts (xy 175.26 125.73) (xy 176.53 125.73))
     (stroke (width 0) (type default))
   )
@@
     (stroke (width 0) (type default))
   )
-  (wire (pts (xy 161.29 78.74) (xy 161.29 81.28))
-    (stroke (width 0) (type default))
-  )
-  (wire (pts (xy 130.81 93.98) (xy 130.81 96.52))
-    (stroke (width 0) (type default))
-  )
   (wire (pts (xy 77.47 143.51) (xy 146.05 143.51))
     (stroke (width 0) (type default))
   )
-  (wire (pts (xy 130.81 81.28) (xy 130.81 83.82))
+  (wire (pts (xy 161.29 71.12) (xy 163.83 71.12))
     (stroke (width 0) (type default))
   )
@@
     (stroke (width 0) (type default))
   )
-  (wire (pts (xy 161.29 91.44) (xy 161.29 93.98))
-    (stroke (width 0) (type default))
-  )
-  (wire (pts (xy 161.29 76.2) (xy 161.29 78.74))
-    (stroke (width 0) (type default))
-  )
   (wire (pts (xy 77.47 143.51) (xy 77.47 41.91))
     (stroke (width 0) (type default))
   )
-  (wire (pts (xy 130.81 60.96) (xy 130.81 63.5))
-    (stroke (width 0) (type default))
-  )
   (wire (pts (xy 172.72 68.58) (xy 172.72 113.03))
     (stroke (width 0) (type default))
   )
-  (wire (pts (xy 161.29 93.98) (xy 161.29 96.52))
-    (stroke (width 0) (type default))
-  )
-  (wire (pts (xy 130.81 68.58) (xy 130.81 71.12))
-    (stroke (width 0) (type default))
-  )
-  (wire (pts (xy 146.05 48.26) (xy 130.81 48.26))
-    (stroke (width 0) (type default))
-  )
-  (wire (pts (xy 130.81 73.66) (xy 130.81 76.2))
-    (stroke (width 0) (type default))
-  )
-  (wire (pts (xy 161.29 121.92) (xy 97.79 121.92))
-    (stroke (width 0) (type default))
-  )
-  (wire (pts (xy 161.29 88.9) (xy 161.29 91.44))
-    (stroke (width 0) (type default))
-  )
-  (wire (pts (xy 130.81 63.5) (xy 130.81 66.04))
-    (stroke (width 0) (type default))
-  )
-  (wire (pts (xy 161.29 71.12) (xy 161.29 73.66))
+  (wire (pts (xy 127 48.26) (xy 146.05 48.26))
     (stroke (width 0) (type default))
   )
@@
     (stroke (width 0) (type default))
   )
-  (wire (pts (xy 161.29 86.36) (xy 161.29 88.9))
-    (stroke (width 0) (type default))
-  )
   (wire (pts (xy 148.59 158.75) (xy 168.91 158.75))
     (stroke (width 0) (type default))
   )
-  (wire (pts (xy 130.81 76.2) (xy 130.81 78.74))
-    (stroke (width 0) (type default))
-  )
-  (wire (pts (xy 130.81 58.42) (xy 130.81 60.96))
-    (stroke (width 0) (type default))
-  )
   (wire (pts (xy 237.49 49.53) (xy 236.22 49.53))
     (stroke (width 0) (type default))
@@
     (stroke (width 0) (type default))
   )
-  (wire (pts (xy 161.29 73.66) (xy 161.29 76.2))
-    (stroke (width 0) (type default))
-  )
-  (wire (pts (xy 130.81 48.26) (xy 130.81 53.34))
+  (wire (pts (xy 163.83 71.12) (xy 163.83 121.92))
     (stroke (width 0) (type default))
   )
@@
     (stroke (width 0) (type default))
   )
-  (wire (pts (xy 161.29 121.92) (xy 161.29 125.73))
-    (stroke (width 0) (type default))
-  )
   (wire (pts (xy 123.19 82.55) (xy 123.19 118.11))
     (stroke (width 0) (type default))
@@
     (stroke (width 0) (type default))
   )
-  (wire (pts (xy 130.81 88.9) (xy 130.81 91.44))
-    (stroke (width 0) (type default))
-  )
-  (wire (pts (xy 161.29 96.52) (xy 161.29 121.92))
-    (stroke (width 0) (type default))
-  )
   (wire (pts (xy 203.2 120.65) (xy 210.82 120.65))
     (stroke (width 0) (type default))
@@
     (stroke (width 0) (type default))
   )
-  (wire (pts (xy 161.29 83.82) (xy 161.29 86.36))
-    (stroke (width 0) (type default))
-  )
   (wire (pts (xy 189.23 26.67) (xy 189.23 71.12))
     (stroke (width 0) (type default))
   )
-  (wire (pts (xy 130.81 99.06) (xy 130.81 101.6))
+  (wire (pts (xy 161.29 88.9) (xy 171.45 88.9))
     (stroke (width 0) (type default))
   )
@@
     (stroke (width 0) (type default))
   )
-  (wire (pts (xy 130.81 78.74) (xy 130.81 81.28))
-    (stroke (width 0) (type default))
-  )
-  (wire (pts (xy 161.29 81.28) (xy 161.29 83.82))
-    (stroke (width 0) (type default))
-  )
-  (wire (pts (xy 161.29 125.73) (xy 175.26 125.73))
+  (wire (pts (xy 171.45 125.73) (xy 175.26 125.73))
     (stroke (width 0) (type default))
   )
@@
     )
     (pin "1")
+    (pin "2")
     (pin "3")
-    (pin "2")
-    (instances
-      (project "Blinky"
+    (instances
+      (project "Blinky"

Commit message: bugfix
Parts:
- added 100nf: C, symbol Device:C
- added R100: R, symbol Device:R
Connections:
- net VDD: now reaches IC1.3 (VDD), J1.5 (BAT), J2.1 (Pin_1), SW1.1, U1.2 (3V3)
- net VDD: no longer 1k1.1, 2k1.2, ZTS6156.1 (VDD)
- net GND: now reaches J1.1 (TEMP1)
- net GND: now also 2k1.1, IC1.7 (GND), J1.3 (GND_3), J4.5 (GND), U1.1 (GND), U1.26 (GND), U1.42 (GND), U1.43 (GND), ZTS6156.3 (GND), 100nf.2
- net at U1.21 (IO18): now also R100.1
- new net: 100nf.1, R100.2, ZTS6156.1 (VDD)
- new net VCC: 1k1.1, 2k1.2
- now unconnected: J2.2 (Pin_2)
Other:
- moved on the sheet: 1k1, 2k1, IC1, J3, J4

Commit message: bugfix
Parts:
- added C1, C3: 100nf, symbol Device:C
- added VR1: MCP1700x-330xxMB, Package_TO_SOT_SMD:SOT-89-3, symbol Regulator_Linear:MCP1700x-330xxMB
- C2: renamed from 100nf; value C -> 100nf
- R1: renamed from 2k1; value R -> 2k
- R2: renamed from 1k1; value R -> 1k
- R3: renamed from R100; value R -> 100
Connections:
- net GND: now also VR1.1 (GND)
- net VDD: now also C1.1, C1.2, VR1.3 (VO); no longer J1.5 (BAT), J2.1 (Pin_1), SW1.1
- new net: C3.2, J1.5 (BAT), J2.1 (Pin_1), SW1.1
- new net: C3.1, VR1.2 (VI)
Other:
- moved on the sheet: J3

Commit message: bugfix
Parts:
- removed BT1: Battery, symbol Device:Battery
- removed C1: 100nf, symbol Device:C
- added C4 (x2), C5: 100nf, symbol Device:C
Connections:
- net GND: now also C3.2, C4.1, C4.2, C4.2, C5.1; no longer J1.3 (GND_3)
- net VDD: now also C3.1, C4.1
- net at J1.5 (BAT), SW1.1: now also VR1.2 (VI); no longer C3.2, J2.1 (Pin_1)
- net at SW1.2: now also J2.1 (Pin_1)
- net at U1.25 (IO26): now also IC1.5 (IN+); no longer IC1.4 (IN-)
- new net: C5.2, J1.3 (GND_3)
Other:
- moved on the sheet: J2, SW1

Commit message: bugfix
Parts:
- added C6: 1uf, symbol Device:C
- C2, C3, C4, C5: value 100nf -> 1uf
- C7: renamed from C4; value 100nf -> 1uf
Connections:
- net GND: now also C6.1
- net at J1.5 (BAT), SW1.1, VR1.2 (VI): now also C6.2
Changed lines of the file:
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@@
   (junction (at 207.01 96.52) (diameter 0) (color 0 0 0 0)
   )
+  (junction (at 241.3 49.53) (diameter 0) (color 0 0 0 0)
+  )
+  (junction (at 236.22 39.37) (diameter 0) (color 0 0 0 0)
+  )
   (junction (at 209.55 49.53) (diameter 0) (color 0 0 0 0)
   )
@@
   (junction (at 200.66 39.37) (diameter 0) (color 0 0 0 0)
   )
-  (junction (at 236.22 49.53) (diameter 0) (color 0 0 0 0)
+  (junction (at 215.9 49.53) (diameter 0) (color 0 0 0 0)
   )
   (wire (pts (xy 149.86 139.7) (xy 149.86 138.43))
@@
     (stroke (width 0) (type default))
   )
+  (wire (pts (xy 236.22 43.18) (xy 233.68 43.18))
+    (stroke (width 0) (type default))
+  )
+  (wire (pts (xy 236.22 39.37) (xy 236.22 43.18))
+    (stroke (width 0) (type default))
+  )
   (wire (pts (xy 210.82 105.41) (xy 210.82 101.6))
     (stroke (width 0) (type default))
@@
     (stroke (width 0) (type default))
   )
+  (wire (pts (xy 226.06 49.53) (xy 215.9 49.53))
+    (stroke (width 0) (type default))
+  )
   (wire (pts (xy 185.42 82.55) (xy 185.42 87.63))
     (stroke (width 0) (type default))
@@
     (stroke (width 0) (type default))
   )
-  (wire (pts (xy 223.52 49.53) (xy 223.52 39.37))
-    (stroke (width 0) (type default))
-  )
   (wire (pts (xy 185.42 87.63) (xy 207.01 87.63))
     (stroke (width 0) (type default))
@@
     (stroke (width 0) (type default))
   )
+  (wire (pts (xy 241.3 49.53) (xy 251.46 49.53))
+    (stroke (width 0) (type default))
+  )
+  (wire (pts (xy 241.3 39.37) (xy 241.3 49.53))
+    (stroke (width 0) (type default))
+  )
   (wire (pts (xy 97.79 130.81) (xy 96.52 130.81))
     (stroke (width 0) (type default))
@@
     (stroke (width 0) (type default))
   )
+  (wire (pts (xy 226.06 43.18) (xy 226.06 49.53))
+    (stroke (width 0) (type default))
+  )
   (wire (pts (xy 186.69 68.58) (xy 198.12 68.58))
     (stroke (width 0) (type default))
@@
     (stroke (width 0) (type default))
   )
+  (wire (pts (xy 223.52 39.37) (xy 236.22 39.37))
+    (stroke (width 0) (type default))
+  )
   (wire (pts (xy 200.66 39.37) (xy 200.66 45.72))
     (stroke (width 0) (type default))
@@
     (stroke (width 0) (type default))
   )
-  (wire (pts (xy 223.52 49.53) (xy 236.22 49.53))
+  (wire (pts (xy 236.22 39.37) (xy 241.3 39.37))
     (stroke (width 0) (type default))
   )
@@
     (stroke (width 0) (type default))
   )
-  (wire (pts (xy 236.22 49.53) (xy 251.46 49.53))
+  (wire (pts (xy 236.22 49.53) (xy 241.3 49.53))
     (stroke (width 0) (type default))
   )
@@
       (effects (font (size 1.27 1.27)))
     )
-    (property "Value" "100nf" (at 182.88 63.5 90)
+    (property "Value" "1uf" (at 182.88 63.5 90)
       (effects (font (size 1.27 1.27)))
     )
@@
       (effects (font (size 1.27 1.27)))
     )
-    (property "Value" "100nf" (at 134.62 123.19 90)
+    (property "Value" "1uf" (at 134.62 123.19 90)
       (effects (font (size 1.27 1.27)))
     )
@@
       (effects (font (size 1.27 1.27)) (justify right))
     )
-    (property "Value" "100nf" (at 176.53 96.52 0)
+    (property "Value" "1uf" (at 176.53 96.52 0)
       (effects (font (size 1.27 1.27)) (justify right))
     )
@@
     )
   )
+  (symbol (lib_id "Device:C") (at 229.87 43.18 90) (unit 1)
+    (in_bom yes) (on_board yes) (dnp no) (fields_autoplaced)
+    (property "Reference" "C6" (at 229.87 35.56 90)
+      (effects (font (size 1.27 1.27)))
+    )
+    (property "Value" "1uf" (at 229.87 38.1 90)
+      (effects (font (size 1.27 1.27)))
+    )
+    (property "Footprint" "" (at 233.68 42.2148 0)
+      (effects (font (size 1.27 1.27)) hide)
+    )
+    (property "Datasheet" "~" (at 229.87 43.18 0)
+      (effects (font (size 1.27 1.27)) hide)
+    )
+    (pin "1")
+    (pin "2")
+    (instances
+      (project "Blinky"
+        (path "/a854b35b-60aa-44a5-a34e-fbb2d526cb93"
+          (reference "C6") (unit 1)
+        )
+      )
+    )
+  )
   (symbol (lib_id "power:VCC") (at 144.78 139.7 90) (unit 1)
     (in_bom yes) (on_board yes) (dnp no) (fields_autoplaced)
@@
       (effects (font (size 1.27 1.27)))
     )
-    (property "Value" "100nf" (at 205.74 40.64 90)
+    (property "Value" "1uf" (at 205.74 40.64 90)
       (effects (font (size 1.27 1.27)))
     )
@@
   (symbol (lib_id "Device:C") (at 210.82 96.52 90) (unit 1)
     (in_bom yes) (on_board yes) (dnp no) (fields_autoplaced)
-    (property "Reference" "C4" (at 210.82 88.9 90)
-      (effects (font (size 1.27 1.27)))
-    )
-    (property "Value" "100nf" (at 210.82 91.44 90)
+    (property "Reference" "C7" (at 210.82 88.9 90)
+      (effects (font (size 1.27 1.27)))
+    )
+    (property "Value" "1uf" (at 210.82 91.44 90)
       (effects (font (size 1.27 1.27)))
     )
@@
       (project "Blinky"
         (path "/a854b35b-60aa-44a5-a34e-fbb2d526cb93"
-          (reference "C4") (unit 1)
-        )
-      )
+          (reference "C7") (unit 1)
+        )
+      )

Commit message: bugfix
Parts:
- removed C4: 1uf, symbol Device:C
- removed J4: USB_B_Micro, symbol Connector:USB_B_Micro
- removed R1: 2k, symbol Device:R
- removed R2: 1k, symbol Device:R
- added C8, C9: 1uf, symbol Device:C
- added J?: Conn_01x04_Pin, symbol Connector:Conn_01x04_Pin
- added R4: R, symbol Device:R
Connections:
- net GND: now also J2.2 (Pin_2), C9.1, J?.4 (Pin_4), R4.1
- net VDD: now also IC1.2 (PVDD), J?.1 (Pin_1)
- net at J1.2 (PROG2): now also R4.2
- net at U1.25 (IO26): now also C8.1; no longer IC1.5 (IN+)
- net at U1.37 (TXD0): now also J?.2 (Pin_2)
- net at U1.38 (RXD0): now also J?.3 (Pin_3)
- net at IC1.4 (IN-): now also C9.2
- new net: C8.2, IC1.5 (IN+)
Other:
- moved on the sheet: C5

Commit message: beta schematic
Parts:
- removed C7: 1uf, symbol Device:C
- removed U1: ESP32-S2-WROVER, RF_Module:ESP32-S2-WROVER, symbol RF_Module:ESP32-S2-WROVER
- added C1, C5: 1uf, symbol Device:C
- added J1: Conn_01x03_Pin, symbol Connector:Conn_01x03_Pin
- added Q1, Q2, Q3, Q4, Q5, Q6: IRLML6244, Package_TO_SOT_SMD:SOT-23, symbol Transistor_FET:IRLML6244
- added R1, R11, R14, R15, R3, R5, R7, R9: 1, symbol Device:R
- added R10, R12, R2, R4, R6, R8: 100, symbol Device:R
- added U1, U2: XL-HD6070RGBC-A46L, footprint:LED-SMD_XL-HD6070RGBC-A46L, symbol XL-HD6070RGBC-A46L:XL-HD6070RGBC-A46L
- added U3: ESP32-S2-SOLO-2-N4, footprint:WIRELM-SMD_ESP32-S3-WROOM-1, symbol ESP32-S2-SOLO-2-N4:ESP32-S2-SOLO-2-N4
- R16: renamed from R4; value R -> 1
- gave numbers to parts that had none: 1
- renumbered C5 to C3, C9 to C4, C8 to C6, C3 to C7, C6 to C8, J1 to J4, J2 to J6, R3 to R13, ZTS6156 to ZTS1
Connections:
- net GND: now also J4.8 (CE), C1.1, C5.1, J1.1 (Pin_1), Q6.1 (G), R1.2, R11.2, R12.1, R3.2, R5.2, R7.2, R9.2, U1.7, U2.7, U3.41 (GND)
- net VDD: now also C1.2, C5.2, J1.2 (Pin_2), R14.2, R15.2, U1.1, U1.3, U1.5, U2.1, U2.3, U2.5, U3.2 (3V3), U3.3 (EN); no longer IC1.2 (PVDD)
- net at C6.1: now also U3.25 (IO34)
- net at J2.2 (Pin_2): now also U3.36 (RXD0)
- net at J2.3 (Pin_3): now also U3.37 (TXD0)
- net at R13.1: now also U3.10 (IO17)
- net at ZTS1.2 (OUTPUT): now also U3.5 (IO5)
- net at IC1.6 (~{SD}): now also U3.26 (IO45)
- new net: Q3.2 (S), R5.1
- new net: Q6.2 (S), R11.1
- new net: Q6.3 (D), U1.6
- new net: Q4.3 (D), U1.2
- new net: Q5.3 (D), U1.4
- new net: Q1.1 (G), R2.1
- new net: R2.2, U3.17 (IO9)
- new net: Q3.1 (G), R6.1
- new net: R6.2, U3.14 (IO20)
- new net: Q4.1 (G), R8.1
- new net: Q4.2 (S), R7.1
- new net: Q1.2 (S), R1.1
- new net: Q3.3 (D), U2.2
- new net: Q2.3 (D), U2.4
- new net: Q1.3 (D), U2.6
- new net: R12.2, U3.13 (IO19)
- new net: IC1.2 (PVDD), R14.1, R15.1
- new net: Q2.2 (S), R3.1
- new net: Q5.1 (G), R10.1
- new net: Q5.2 (S), R9.1
- new net: J1.3 (Pin_3), U3.27 (IO0)
- new net: Q2.1 (G), R4.1
- new net: R4.2, U3.15 (IO3)
- new net: R10.2, U3.12 (IO8)
- new net: R8.2, U3.11 (IO18)

Commit message: updated Schematic
Parts:
- removed IC1: PAM8303CBSC, SOP65P490X110-8N, symbol PAM8303CBSC:PAM8303CBSC
- removed J4: TP4056, SOIC127P600X175-9N, symbol TP4056:TP4056
- removed ZTS1: Microphone, SPU0414HR5H-SB, symbol SPU0410HR5H-PB:SPU0410HR5H-PB
- added R13, R14, R15, R16, R17, R18: 100k, symbol Device:R
- added U3: ZTS6156, footprint:MIC-SMD_3P-L2.8-W1.9_ZTS6056, symbol ZTS6156:ZTS6156
- added U5: PAM8303DBSC, footprint:MSOP-8_L3.0-W3.0-P0.65-LS5.0-BL, symbol PAM8303DBSC:PAM8303DBSC
- added U6: TP4056_C725790, footprint:ESOP-8_L4.9-W3.9-P1.27-LS6.0-BL-EP, symbol TP4056_C725790:TP4056_C725790
- renumbered J5 to J4, J6 to J5, R13 to R19, R14 to R20, R15 to R21, R16 to R22, U3 to U4
Connections:
- net GND: now also R13.2, R14.2, R15.2, R16.2, R17.2, R18.2, U3.3 (GND), U5.7 (GND), U6.1 (TEMP), U6.8 (CE); no longer Q6.1 (G), R12.1
- net VDD: now also C8.2, SW1.1, VR1.2 (VI), U5.3 (VDD), U6.5 (BAT)
- net at R22.2: now also U6.2 (PROG)
- net at C3.2: now also U6.3 (GND)
- net at C6.2: now also U5.5 (IN+)
- net at C4.2: now also U5.4 (IN-)
- net at R2.2, U4.17 (IO9): now also R14.1
- net at R6.2, U4.14 (IO20): now also R15.1
- net at C2.1, R19.2: now also U4.5 (IO5), U3.1 (VDD), U3.2 (OUT)
- net at R12.2, U4.13 (IO19): now also R16.1
- net at R20.1, R21.1: now also U5.2 (PVDD)
- net at R4.2, U4.15 (IO3): now also R13.1
- net at R10.2, U4.12 (IO8): now also R17.1
- net at R8.2, U4.11 (IO18): now also R18.1
- net at J3.1 (Pin_1): now also U5.1 (OUT+)
- net at J3.2 (Pin_2): now also U5.8 (OUT-)
- net at U4.26 (IO45): now also U5.6 (SD#)
- new net: Q6.1 (G), R12.1
