File: Blinky/Blinky3.kicad_pcb (KiCad board)
At the start: 2 copper layers, 57 parts, among them J1 Conn_01x04_Pin, J2 Conn_01x03_Pin, J3 Battery Connector, J4 Charging Notches, J5 Speaker Connector, Q1 IRLML6244, Q2 IRLML6244, Q3 IRLML6244, Q4 IRLML6244, Q5 IRLML6244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

Commit message: updated pcb layout
Parts:
- C5, C8, Q1, Q2, Q3, R1, R13, R14, R15, R2, R3, R4, R5, R6, U6, U7: moved to B.Cu
- moved R25 5.52 mm to (130.9, 81.0)
- moved R4 5.09 mm to (146.9, 71.0)
- moved R14 2.51 mm to (150.3, 70.8), turned to 180 degrees
- moved R1 1.75 mm to (146.8, 69.5)
- moved R2 1.50 mm to (146.8, 67.8)
- moved U8 1.50 mm to (164.6, 76.5), turned to 0 degrees
- moved J4 1.33 mm to (160.4, 47.8), turned to 0 degrees
- moved R20 1.15 mm to (161.7, 83.2)
- moved U7 0.42 mm to (131.1, 82.2), turned to 180 degrees
- moved Q1 0.40 mm to (150.5, 67.8)
- moved R5 0.40 mm to (156.0, 60.2)
- moved U2 0.32 mm to (152.0, 54.0)
- moved Q2 0.25 mm to (150.5, 64.0)
- moved C5 0.20 mm to (131.2, 88.5)
- moved C9 0.10 mm to (131.0, 77.0)
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Connections:
- C10 pad 2: VBAT -> VDD
- C3 pad 2: VBAT -> VDD
- C4 pad 2: VBAT -> VDD
- R21 pad 2: VBAT -> VDD
- SW1 pad 2: VBAT -> VDD
- U1 pad 1: VBAT -> VDD
- U1 pad 3: VBAT -> VDD
- U1 pad 5: VBAT -> VDD
- U2 pad 1: VBAT -> VDD
- U2 pad 3: VBAT -> VDD
- U2 pad 5: VBAT -> VDD
- U6 pad 5: VBAT -> VDD
- U7 pad 2: VBAT -> VDD
- U7 pad 3: VBAT -> VDD
- U8 pad 2: VBAT -> VDD
Routing:
- net VBAT: track 127.5 -> 0.00 mm, vias 7 -> 0
- net /BAT+: track 59.7 -> 0.00 mm, vias 4 -> 0
- net GND: track 254.4 -> 198.3 mm, vias 22 -> 16
- net Net-(Q2-S): track 12.4 -> 4.42 mm, vias 0 -> 2
- net Net-(Q2-D): track 13.1 -> 5.45 mm, vias 3 -> 0
- net VDD: track 167.6 -> 160.2 mm, vias 11 -> 10
- net Net-(Q2-G): track 8.22 -> 13.6 mm, vias 2 -> 0
- net Net-(C9-Pad2): track 11.9 -> 6.65 mm
- net /BLUE2: track 44.9 -> 40.1 mm, vias 2 -> 1
- net Net-(U4-VDD): track 9.05 -> 4.31 mm
- net Net-(U6-CHRG#): track 12.6 -> 9.04 mm, vias 2 -> 1
- net Net-(Q3-G): track 2.56 -> 5.92 mm
- net Net-(J5-Pin_1): track 22.3 -> 25.6 mm, vias 0 -> 1
- net Net-(J5-Pin_2): track 28.6 -> 31.2 mm
- net /RED2: track 36.3 -> 33.9 mm, vias 4 -> 5
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