File: Blinky/Blinky.kicad_pcb (KiCad board)
At the start: 2 copper layers, 57 parts, among them J1 Conn_01x04_Pin, J2 Conn_01x03_Pin, J3 Battery Connector, J4 Charging Notches, J5 Speaker Connector, Q1 IRLML6244, Q2 IRLML6244, Q3 IRLML6244, Q4 IRLML6244, Q5 IRLML6244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

Commit message: updated pcb
Parts:
- moved R6 0.35 mm to (154.9, 67.1)
- moved R4 0.07 mm to (151.9, 71.4)
Connections:
- J4 pad 1: VDD -> CHARGE+
- U10 pad 2: VDD -> CHARGE+
- U6 pad 4: VDD -> CHARGE+
- U6 pad 8: VDD -> CHARGE+
- U9 pad 2: VDD -> CHARGE+
Routing:
- net VDD: track 167.6 -> 114.0 mm, vias 11 -> 6
- net CHARGE+: track 0.00 -> 41.5 mm, vias 0 -> 4
- net GND: track 254.4 -> 250.8 mm
- net Net-(U9-K): track 5.26 -> 8.53 mm, vias 0 -> 2
- net Net-(J5-Pin_2): track 28.6 -> 27.2 mm, vias 1 -> 0
- net /SOUND_ENABLE: vias 1 -> 0

Commit message: updated pcb
Parts:
- moved R6 0.16 mm to (155.0, 67.2)
Routing:
- net VDD: track 114.0 -> 159.4 mm, vias 6 -> 9
- net GND: track 250.8 -> 271.4 mm, vias 22 -> 23
- net /RED2: track 36.3 -> 35.7 mm
- net Net-(Q3-G): track 2.56 -> 3.08 mm
Other:
- board outline added: 40.1 x 64.6 mm

Commit message: updated pcb
Parts:
- J4: footprint Connector_PinHeader_1.00mm:PinHeader_1x02_P1.00mm_Horizontal -> Library:ChargingNotches
- moved J3 7.00 mm to (163.0, 107.0)
- moved J4 5.47 mm to (156.3, 44.3), turned to 180 degrees
- moved U8 1.24 mm to (163.9, 76.0)
- moved C4 0.74 mm to (162.7, 87.3)
Routing:
- net GND: track 271.4 -> 302.3 mm, vias 23 -> 77
- net /BAT-: track 5.68 -> 13.5 mm, vias 0 -> 2
- net Net-(Q6-D): track 20.0 -> 16.4 mm
- net /BAT+: track 59.7 -> 63.3 mm
- net CHARGE+: track 41.5 -> 44.7 mm
- net Net-(Q5-D): track 21.1 -> 18.3 mm
- net /GREEN1: track 55.0 -> 53.9 mm
- net unconnected-(U3-IO15-Pad8): track 1.00 -> 0.00 mm
- net /RED1: track 58.5 -> 57.7 mm
- net VDD: track 159.4 -> 159.0 mm, vias 9 -> 10
- added copper zone on B.Cu, net GND
- added copper zone on F.Cu, net GND

Commit message: updated pcb
Parts:
- moved J3 1.85 mm to (163.0, 105.2)
- moved C2 0.78 mm to (161.0, 102.0)
Routing:
- net /BAT+: track 63.3 -> 61.5 mm
- net GND: track 302.3 -> 303.2 mm
- net /BAT-: track 13.5 -> 12.7 mm

Commit message: updated pcb layout
Parts:
- J5: footprint Connector_JST:JST_PH_B2B-PH-K_1x02_P2.00mm_Vertical -> footprint:CONN-TH_B2B-PH-K-S
- R5, R7: value 1 -> 2
- U5: value ~ -> XB4908A
- U8: value HT7533-1_C14289 -> HT7833-A
- moved J5 1.50 mm to (131.5, 105.1), turned to 0 degrees
Connections:
- R21 pad 2: VBAT -> /BAT+
- U6 pad 5: VBAT -> /BAT+
Routing:
- net VBAT: track 127.5 -> 116.8 mm
- net /BAT+: track 61.5 -> 69.8 mm, vias 4 -> 5
- net GND: track 303.2 -> 301.0 mm

Commit message: newest version
Parts:
- moved J5 0.57 mm to (131.1, 104.7), turned to -90 degrees
Routing:
- net Net-(J5-Pin_2): track 26.7 -> 25.5 mm
- net Net-(J5-Pin_1): track 22.1 -> 23.2 mm
Changed lines of the file:
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@@
   )
   (footprint "footprint:CONN-TH_B2B-PH-K-S" (layer "F.Cu")
-    (at 131.5 105.1)
+    (at 131.1 104.7 -90)
     (descr "CONN-TH_B2B-PH-K-S footprint")
     (tags "CONN-TH_B2B-PH-K-S footprint")
@@
     (property "ki_keywords" "connector")
     (attr through_hole)
-    (fp_text reference "J5" (at 0.039522 -4.159004) (layer "F.SilkS")
-        (effects (font (size 1 1) (thickness 0.15)))
-    )
-    (fp_text value "Speaker Connector" (at 0.039522 3.651003) (layer "F.Fab")
-        (effects (font (size 1 1) (thickness 0.15)))
-    )
-    (fp_text user "REF**" (at 0.039522 5.651003) (layer "F.Fab")
+    (fp_text reference "J5" (at 0.039522 -4.159004 90) (layer "F.SilkS")
+        (effects (font (size 1 1) (thickness 0.15)))
+    )
+    (fp_text value "Speaker Connector" (at 0.039522 3.651003 90) (layer "F.Fab")
+        (effects (font (size 1 1) (thickness 0.15)))
+    )
+    (fp_text user "REF**" (at 0.039522 5.651003 90) (layer "F.Fab")
         (effects (font (size 1 1) (thickness 0.15)))
     )
@@
     (fp_circle (center 2.950013 -2.8) (end 2.98001 -2.8)
       (stroke (width 0.059995) (type solid)) (fill none) (layer "F.SilkS"))
-    (pad "1" thru_hole circle (at 1 0) (size 1.6 1.6) (drill 0.900025) (layers "*.Cu" "*.Mask")
+    (pad "1" thru_hole circle (at 1 0 270) (size 1.6 1.6) (drill 0.900025) (layers "*.Cu" "*.Mask")
       (net 6 "Net-(J5-Pin_1)") (pinfunction "Pin_1") (pintype "passive"))
-    (pad "2" thru_hole circle (at -1 0) (size 1.6 1.6) (drill 0.900025) (layers "*.Cu" "*.Mask")
+    (pad "2" thru_hole circle (at -1 0 270) (size 1.6 1.6) (drill 0.900025) (layers "*.Cu" "*.Mask")
       (net 34 "Net-(J5-Pin_2)") (pinfunction "Pin_2") (pintype "passive"))
     (model "/Users/julian/Code/sparkles/JLC2KiCad_lib/footprint/packages3d/CONN-TH_B2B-PH-K-S.wrl"
@@
   (segment (start 130.475 88.3) (end 131.55 87.225) (width 0.25) (layer "F.Cu") (net 5))
   (segment (start 132.175 87.225) (end 132.325 87.075) (width 0.25) (layer "F.Cu") (net 5))
+  (segment (start 132.4 103.4) (end 132.4 104.4) (width 0.25) (layer "F.Cu") (net 6))
+  (segment (start 132.4 104.4) (end 131.1 105.7) (width 0.25) (layer "F.Cu") (net 6))
+  (segment (start 129.25 100.25) (end 132.4 103.4) (width 0.25) (layer "F.Cu") (net 6))
+  (segment (start 130.324892 84.74605) (end 129.25 85.820942) (width 0.25) (layer "F.Cu") (net 6))
   (segment (start 129.25 85.820942) (end 129.25 100.25) (width 0.25) (layer "F.Cu") (net 6))
-  (segment (start 130.324892 84.74605) (end 129.25 85.820942) (width 0.25) (layer "F.Cu") (net 6))
-  (segment (start 129.25 100.25) (end 132.5 103.5) (width 0.25) (layer "F.Cu") (net 6))
-  (segment (start 132.5 103.5) (end 132.5 105.1) (width 0.25) (layer "F.Cu") (net 6))
   (segment (start 147.575 69.25) (end 150.8875 69.25) (width 0.25) (layer "F.Cu") (net 7))
   (segment (start 147.575 67.75) (end 148.125 67.2) (width 0.25) (layer "F.Cu") (net 8))
@@
   (segment (start 163 100.452208) (end 163 103.6) (width 0.2) (layer "B.Cu") (net 33))
   (segment (start 163.05 105.35) (end 163 105.4) (width 0.2) (layer "B.Cu") (net 33))
-  (segment (start 128.8 102.8) (end 130.5 104.5) (width 0.25) (layer "F.Cu") (net 34))
+  (segment (start 128.8 101.4) (end 131.1 103.7) (width 0.25) (layer "F.Cu") (net 34))
+  (segment (start 130.324892 80.45395) (end 129.14605 80.45395) (width 0.25) (layer "F.Cu") (net 34))
+  (segment (start 128.8 80.8) (end 128.8 101.4) (width 0.25) (layer "F.Cu") (net 34))
   (segment (start 129.14605 80.45395) (end 128.8 80.8) (width 0.25) (layer "F.Cu") (net 34))
-  (segment (start 130.324892 80.45395) (end 129.14605 80.45395) (width 0.25) (layer "F.Cu") (net 34))
-  (segment (start 130.5 104.5) (end 130.5 105.1) (width 0.25) (layer "F.Cu") (net 34))
-  (segment (start 128.8 80.8) (end 128.8 102.8) (width 0.25) (layer "F.Cu") (net 34))
   (segment (start 145.925 69.825) (end 145.5 70.25) (width 0.25) (layer "F.Cu") (net 35))
   (segment (start 133.75 72.25) (end 135.75 72.25) (width 0.25) (layer "F.Cu") (net 35))
