File: Blinky/_autosave-Blinky.kicad_sch (KiCad schematic)
At the start: 60 parts, among them J1 Conn_01x06_Socket, J2 Conn_01x06_Socket, J3 Battery Connector, J4 Charging Notches, Q1 IRLML6244, Q2 IRLML6244, Q3 IRLML6244, Q4 IRLML6244, Q5 IRLML6244, Q6 IRLML6244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

Commit message: version 1.95
Parts:
- gave numbers to parts that had none: 1
Changed lines of the file:
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@@
   (symbol (lib_id "MICROXNJ:MICROXNJ") (at 280.67 80.01 0) (unit 1)
     (in_bom yes) (on_board yes) (dnp no) (fields_autoplaced)
-    (property "Reference" "USB?" (at 289.56 78.74 0)
+    (property "Reference" "USB1" (at 289.56 78.74 0)
       (effects (font (size 1.27 1.27)) (justify left))
     )
@@
       (project "Blinky"
         (path "/a854b35b-60aa-44a5-a34e-fbb2d526cb93"
-          (reference "USB?") (unit 1)
+          (reference "USB1") (unit 1)
         )
       )

Commit message: trying to fix C5
Parts:
- removed R19: 10k, Resistor_SMD:R_0603_1608Metric, symbol Device:R
- removed R24: 1k, Resistor_SMD:R_0603_1608Metric, symbol Device:R
- removed U4: LM358_C5296727, footprint:SO-8_L4.9-W3.9-P1.27-LS6.0-BL, symbol LM358_C5296727:LM358_C5296727
- removed U8: HT7833-A, otherfootprint:SOT-89-3_L4.5-W2.5-P1.50-LS4.2-BR, symbol HT7533-1_C14289:HT7533-1_C14289
- added C11: 1uF, Capacitor_SMD:C_0603_1608Metric, symbol Device:C
- added C5: 1000uf, footprint:CAP-SMD_BD8.0-L8.3-W8.3-FD, symbol Device:C
- added C9: 1uf, Capacitor_SMD:C_0603_1608Metric, symbol Device:C
- added R30, R31, R33: 100k, Resistor_SMD:R_0603_1608Metric, symbol Device:R
- added R32: 470R, Resistor_SMD:R_0603_1608Metric, symbol Device:R
- added R34: 10k, Resistor_SMD:R_0603_1608Metric, symbol Device:R
- added U13, U14: XL-HD6070RGBC-A46L, footprint:LED-SMD_XL-HD6070RGBC-A46L-BACKSIDE, symbol XL-HD6070RGBC-A46L:XL-HD6070RGBC-A46L
- added U15: TS-1187A-B-A-B, footprint:SW-SMD_4P-L5.1-W5.1-P3.70-LS6.5-TL-2, symbol TS-1187A-B-A-B:TS-1187A-B-A-B
- added U4: TLV9002IDR, footprint:SOIC-8_L4.9-W3.9-P1.27-LS6.0-BL, symbol TLV9002IDR:TLV9002IDR
- added U8: ME6217C33M5G, footprint:SOT-23-5_L3.0-W1.7-P0.95-LS2.8-BR, symbol ME6217C33M5G:ME6217C33M5G
- C1: value 1uf -> 47uf
- C2: value 220nf -> 100pF optional
- C4: value 100nf -> 470nF
- C6: value 100uF -> 10uf
- C8: value 1uf -> 100nf
- R1, R11: value 1 -> 4
- R25: value 10k -> 100k
- R26: value 1k -> 47k
- R28: value 100k -> 10k
- R5, R7: value 2 -> 1
Connections:
- net BLUE1: now also R18.2, R8.2, U3.11 (IO18); no longer R12.2, R16.2
- net BLUE2: now also R15.2, R6.2, U3.30 (IO37); no longer R13.2, R2.2, U3.17 (IO9)
- net GND: now also C3.2, J2.6 (Pin_6), C11.2, C5.2, C9.1, U15.3 (C), U4.4 (V-), U8.2 (VSS); no longer C3.1, R28.2, U1.7, U2.7
- net MIC: now also R25.1, U4.1 (OUT1); no longer C2.1
- net RED1: now also R12.2, R16.2, U3.31 (IO38); no longer R18.2, R8.2, U3.11 (IO18)
- net RED2: now also R13.2, R2.2, U3.17 (IO9); no longer R15.2, R6.2
- net VBAT: now also J2.1 (Pin_1), U8.1 (VIN), U8.3 (CE)
- net VDD: now also C5.1, R30.1, R31.1, R32.1, R33.2, U4.8 (V+), U8.5 (VOUT); no longer C3.2, R29.2, U3.3 (EN)
- net at R27.2: now also C2.1, R34.2, U4.7 (OUT2)
- net at R25.2: now also R34.1, U4.2 (IN1-); no longer R26.2
- net at R27.1, R28.1: now also C2.2, U4.6 (IN2-); no longer C4.1
- net at C4.2, U7.1 (+): now also R29.2; no longer R29.1
- net at U11.2 (B): now also R31.2
- net PIN32: now reaches J1.2 (Pin_2)
- net PIN32: now also U3.32 (IO39)
- net PIN33: now reaches J1.3 (Pin_3)
- net PIN33: now also U3.33 (IO40)
- net PIN34: now reaches J1.4 (Pin_4)
- net PIN34: now also U3.34 (IO41)
- net PIN35: now reaches J1.5 (Pin_5)
- net PIN35: now also U3.35 (IO42)
- net PIN9: now reaches J2.2 (Pin_2)
- net PIN9: now also U3.9 (IO16)
- net PIN8: now reaches J2.3 (Pin_3)
- net PIN8: now also U3.8 (IO15)
- net PIN7: now reaches J2.4 (Pin_4)
- net PIN7: now also U3.7 (IO7)
- net PIN6: now reaches J2.5 (Pin_5)
- net PIN6: now also U3.6 (IO6)
- net PIN10: now reaches U3.10 (IO17)
- new net: C11.1, R29.1, R32.2
- new net: C4.1, R28.2
- new net: C9.2, R30.2, U15.2 (B)
- new net EN: U15.1 (A), U3.3 (EN)
- new net VDD_REF: C3.1, R26.2, R33.1, U4.3 (IN1+), U4.5 (IN2+)
Other:
- moved on the sheet: C3, C4, R25, R26, R27, R28, R29, U11, U7
