File: Blinky/_autosave-Blinky.kicad_pcb (KiCad board)
At the start: 4 copper layers, 44.9 x 64.5 mm, 76 parts, among them J1 Conn_01x06_Socket, J2 Conn_01x06_Socket, J3 Battery Connector, J4 Charging Notches, J5 Battery Connector, Q1 IRLML6244, Q2 IRLML6244, Q3 IRLML6244, Q4 IRLML6244, Q5 IRLML6244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

Commit message: updated board
Parts:
- moved U5 4.99 mm to (162.4, 92.6), turned to 90 degrees
Routing:
- net Net-(U4B-IN2-): track 6.77 -> 45.8 mm, vias 1 -> 2
- net Net-(U4B-OUT2): track 8.73 -> 42.2 mm, vias 1 -> 2
- net Net-(Q2-G): track 6.69 -> 29.8 mm, vias 2 -> 4
- net GND: track 70.2 -> 80.7 mm, vias 52 -> 62
- net /PIN6: track 21.8 -> 25.7 mm
- net VDD: track 19.2 -> 23.0 mm, vias 9 -> 11
- net /BAT-: track 19.8 -> 23.1 mm
- net Net-(U5-VDD): track 16.2 -> 17.6 mm
- net /PIN7: track 23.5 -> 24.4 mm
- net /PIN9: track 26.3 -> 25.6 mm
- removed copper zone on B.Cu, net GND
Other:
- board size 44.9 x 64.5 mm -> 44.7 x 64.6 mm
